File: ManipulatorER_v3.kicad_pcb (KiCad board)
At the start: 2 copper layers, 133.3 x 76.2 mm, 22 parts, among them J1 DB15_Female_MountingHoles, J1001 Conn_02x02_Counter_Clockwise, J3 Conn_01x04, J5 Conn_01x02, J6 Conn_01x04, P1 Digital, P2 Power, P3 Analog, P4 Analog, P5 PWM, P6 PWM, P7 Communication, U1 TSR 1-245, U2 TSR 1-243

Commit message: payload pcb v2.0
Parts:
- removed C2: C, Ele Caps:UCM1H220MCL1GS
- removed locked: Conn_01x02, Connector_Molex:Molex_Mega-Fit_76829-0102_2x01_P5.70mm_Vertical
- added C4: 0.1u, Ceramic:C1206C104J4RAC7800, F.Cu at (146.1, 109.3)
- added D1: LED, LED_SMD:LED_0805_2012Metric_Pad1.15x1.40mm_HandSolder, F.Cu at (107.5, 57.0)
- added D2: LED, LED_SMD:LED_0805_2012Metric_Pad1.15x1.40mm_HandSolder, F.Cu at (107.5, 60.0)
- added D3: LED, LED_SMD:LED_0805_2012Metric_Pad1.15x1.40mm_HandSolder, F.Cu at (107.5, 63.0)
- added D4: LED, LED_SMD:LED_0805_2012Metric_Pad1.15x1.40mm_HandSolder, F.Cu at (107.5, 66.0)
- added D5: LED, LED_SMD:LED_0805_2012Metric_Pad1.15x1.40mm_HandSolder, F.Cu at (109.5, 106.4)
- added D6: LED, LED_SMD:LED_0805_2012Metric_Pad1.15x1.40mm_HandSolder, F.Cu at (121.7, 110.0)
- added D7: LED, LED_SMD:LED_0805_2012Metric_Pad1.15x1.40mm_HandSolder, F.Cu at (155.7, 115.8)
- added G***: LOGO, Graphics:Flying_WV_Logo, F.Cu at (158.8, 59.8)
- added J10: Conn_01x15_Male, 5x15Conn:SAMTEC_TSW-105-08-G-T-RA, F.Cu at (228.6, 60.9)
- added J11: Conn_01x04, ConnectorMolex1x4:MOLEX_530480410, F.Cu at (231.2, 88.9)
- added J12: Conn_01x02, Connector_PinHeader_2.54mm:PinHeader_1x02_P2.54mm_Vertical, F.Cu at (111.6, 92.3)
- added J13: Conn_01x04, ConnectorMolex1x4:MOLEX_530480410, F.Cu at (231.2, 99.9)
- added J14: Conn_02x04_Odd_Even, Connector_PinHeader_2.54mm:PinHeader_2x04_P2.54mm_Vertical_SMD, F.Cu at (115.5, 52.2)
- added J15: Conn_01x02, Connector_PinHeader_2.54mm:PinHeader_1x02_P2.54mm_Vertical_SMD_Pin1Right, F.Cu at (128.0, 50.1)
- added J16: Conn_01x02, Connector_Molex:Molex_Mega-Fit_76825-0002_2x01_P5.70mm_Horizontal, F.Cu at (119.2, 72.0)
- added J19: Conn_02x02_Odd_Even, Connector_PinHeader_2.54mm:PinHeader_2x02_P2.54mm_Vertical, F.Cu at (221.5, 86.8)
- added J2: Conn_01x02, Connector_Molex:Molex_Mega-Fit_76825-0002_2x01_P5.70mm_Horizontal, F.Cu at (127.8, 106.0)
- added J4: Conn_01x04, ConnectorMolex1x4:MOLEX_530480410, F.Cu at (231.2, 110.9)
- added J7: Conn_01x02, Connector_Molex:Molex_Mega-Fit_76825-0002_2x01_P5.70mm_Horizontal, F.Cu at (140.0, 106.0)
- added J8: Conn_01x02, Connector_PinHeader_2.54mm:PinHeader_1x02_P2.54mm_Vertical, F.Cu at (111.6, 96.1)
- added J9: Conn_01x15_Male, 5x15Conn:SAMTEC_TSW-105-08-G-T-RA, F.Cu at (228.6, 74.5)
- added R1: 3000, Resistor_SMD:R_0805_2012Metric_Pad1.20x1.40mm_HandSolder, F.Cu at (109.5, 102.1)
- added R2: 750, Resistor_SMD:R_0805_2012Metric_Pad1.20x1.40mm_HandSolder, F.Cu at (121.7, 105.4)
- added R3: 150, Resistor_SMD:R_0805_2012Metric_Pad1.20x1.40mm_HandSolder, F.Cu at (155.7, 112.0)
- added R4: 976, Resistor_SMD:R_0805_2012Metric_Pad1.20x1.40mm_HandSolder, F.Cu at (112.0, 65.0)
- C1: value C -> 0.1u
- C3: value C -> 22u
- J3: value Conn_01x04 -> Conn_01x02; footprint Connector_PinSocket_2.54mm:PinSocket_1x04_P2.54mm_Vertical -> Connector_Molex:Molex_Micro-Fit_3.0_43045-0200_2x01_P3.00mm_Horizontal
- J6: footprint Connector_Molex:Molex_Micro-Fit_3.0_43045-0400_2x02_P3.00mm_Horizontal -> ConnectorMolex1x4:MOLEX_530480410
- U2: value TSR 1-243 -> HTSSOP16_STM; footprint TS Regulators:TSR 1-2433 -> LED_IC:LED8102SXTTR
- moved C1 67.4 mm to (133.9, 109.3), turned to 90 degrees
- moved U2 52.8 mm to (120.4, 63.0), turned to 180 degrees
- moved J1 47.8 mm to (198.9, 111.5), turned to 0 degrees
- moved J3 28.8 mm to (162.1, 112.7), turned to 180 degrees
- moved C3 17.3 mm to (150.9, 114.0), turned to -90 degrees
- moved U1 16.7 mm to (151.5, 108.0)
- moved J6 13.9 mm to (217.6, 117.3), turned to 0 degrees
- moved J5 9.02 mm to (115.6, 105.9)
- moved J17 2.48 mm to (119.2, 86.3)
- moved P1 1.53 mm to (212.3, 91.8)
- moved P2 1.53 mm to (146.3, 96.9)
- moved P3 1.53 mm to (169.2, 96.9)
- moved P4 1.53 mm to (192.0, 96.9)
- moved P5 1.53 mm to (137.2, 48.6)
- moved P6 1.53 mm to (164.1, 48.6)
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- renumbered J1001 to J17
Connections:
- net /SCL renamed /1
- net /SDA renamed /2
- C1 pad 2: /12V -> 12V
- C3 pad 1: 40V -> 12V
- J1 pad 11: A11 -> A12
- J1 pad 12: A13 -> A10
- J1 pad 13: A15 -> A5
- J1 pad 4: A12 -> A11
- J1 pad 5: A14 -> A9
- J17 pad 4: /12V -> 12V
- J3 pad 1: 14(Tx3) -> GND
- J3 pad 2: 15(Rx3) -> +5V
- J6 pad 3: 27 -> 20(SDA)
- J6 pad 4: 29 -> 21(SCL)
- P1 pad 10: /47 -> 47
- P1 pad 11: /44 -> 44
- P1 pad 12: /45 -> 45
- P1 pad 13: /42 -> 42
- P1 pad 14: /43 -> 43
- P1 pad 15: /40 -> 40
- P1 pad 16: /41 -> 41
- P1 pad 18: /39 -> 39
- P1 pad 20: /37 -> 37
- P1 pad 23: /32 -> 32
- P1 pad 26: /31 -> 31
- P1 pad 3: /52(SCK) -> 52(SCK)
- P1 pad 32: /25 -> 25
- P1 pad 34: /23 -> 23
- P1 pad 35: unconnected-(P1-Pad35) -> (no net)
- P1 pad 36: unconnected-(P1-Pad35) -> (no net)
- P1 pad 4: /53(SS) -> 53(SS)
- P1 pad 5: /50(MISO) -> 50(MISO)
- P1 pad 6: /51(MOSI) -> 51(MOSI)
- P1 pad 8: /49 -> 49
- P1 pad 9: /46 -> 46
- P2 pad 1: unconnected-(P2-Pad1) -> (no net)
- P2 pad 4: unconnected-(P2-Pad4) -> 3V3
- P2 pad 5: unconnected-(P2-Pad5) -> (no net)
- P2 pad 8: /Vin -> +5V
- P3 pad 6: /A5 -> A5
- P4 pad 2: /A9 -> A9
- P4 pad 3: /A10 -> A10
- P4 pad 6: A13 -> /A13
- P4 pad 7: A14 -> /A14
- P4 pad 8: A15 -> /A15
- P5 pad 8: /10(**) -> 10(**)
- P5 pad 9: /9(**) -> 9(**)
- P6 pad 1: /7(**) -> 7(**)
- P6 pad 7: /1(Tx0) -> 1(Tx0)
- P6 pad 8: /0(Rx0) -> 0(Rx0)
- P7 pad 1: 14(Tx3) -> /14(Tx3)
- P7 pad 2: 15(Rx3) -> /15(Rx3)
- P7 pad 3: /16(Tx2) -> 16(Tx2)
- P7 pad 4: /17(Rx2) -> 17(Rx2)
- P7 pad 7: /20(SDA) -> 20(SDA)
- P7 pad 8: /21(SCL) -> 21(SCL)
- U1 pad 1: 40V -> 12V
- U2 pad 1: 40V -> GND
- U2 pad 2: GND -> 49
- U2 pad 3: 3V3 -> 47
Routing:
- net /+7V: track 0.00 -> 122.2 mm, vias 0 -> 4
- net 47: track 0.00 -> 113.6 mm, vias 0 -> 2
- net 49: track 0.00 -> 112.8 mm, vias 0 -> 2
- net 1(Tx0): track 0.00 -> 106.3 mm, vias 0 -> 7
- net 15(Rx3): track 101.6 -> 0.00 mm, vias 2 -> 0
- net 14(Tx3): track 97.1 -> 0.00 mm, vias 2 -> 0
- net +5V: track 105.4 -> 19.2 mm
- net 16(Tx2): track 0.00 -> 83.9 mm, vias 0 -> 3
- net 10(**): track 0.00 -> 81.1 mm, vias 0 -> 2
- net 17(Rx2): track 0.00 -> 80.1 mm, vias 0 -> 3
- net 7(**): track 0.00 -> 79.3 mm, vias 0 -> 3
- net /12V: track 79.0 -> 0.00 mm
- net 20(SDA): track 0.00 -> 78.2 mm
- net 0(Rx0): track 0.00 -> 78.0 mm, vias 0 -> 1
- net 21(SCL): track 0.00 -> 77.8 mm
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- added copper zone on F.Cu, net 12V
- added copper zone on F.Cu, net Vmisc
Other:
- board text added: "12V"
- board text added: "12V 40V"
- board text added: "40V"
- board text added: "5 V"
- board text added: "5V"
- board text added: "5V Regulator"
- board text added: "ASTRO Payload PCB V2.0"
- board text added: "Analog Input"
- board text added: "Authors: Michael Butts, Zach Waddell, Kendra Gillo"
- board text added: "Digital IO 1"
- board text added: "Digital IO 2"
- board text added: "Digital IO 3"
- board text added: "Fan 1"
- board text added: "Fan 2"
- board text added: "GND"
- board text added: "I2C"
- board text added: "LED controller"
- board text added: "Motor Controls"
- board text added: "Rx"
- board text added: "Tx"
- board text added: "University Rover Challenge 2021-2022"
- board text added: "Vmisc"
- board text added: "Vmisc/5V"
