File: ManipulatorER_v3.kicad_sch (KiCad schematic)
At the start: 22 parts, among them J1 DB15_Female_MountingHoles, J1001 Conn_02x02_Counter_Clockwise, J3 Conn_01x04, J4 Conn_01x02, J5 Conn_01x02, J6 Conn_01x04, P1 Digital, P2 Power, P3 Analog, P4 Analog, P5 PWM, P6 PWM, P7 Communication, U1 TSR 1-245, U2 TSR 1-243

Commit message: payload pcb v2.0
Parts:
- removed C2: 22u, Ele Caps:UCM1H220MCL1GS, symbol Device:C
- removed J3: Conn_01x04, Connector_PinSocket_2.54mm:PinSocket_1x04_P2.54mm_Vertical, symbol Connector_Generic:Conn_01x04
- removed J4: Conn_01x02, Connector_Molex:Molex_Mega-Fit_76829-0102_2x01_P5.70mm_Vertical, symbol Connector_Generic:Conn_01x02
- removed U2: TSR 1-243, TS Regulators:TSR 1-2433, symbol Regulators:173010342
- added C4: 0.1u, ManipulatorER_V3:C1206C104J4RAC7800, symbol Device:C
- added D1, D2, D3, D4, D5, D6, D7: LED, LED_SMD:LED_0805_2012Metric_Pad1.15x1.40mm_HandSolder, symbol Device:LED
- added J10, J9: Conn_01x15_Male, ManipulatorER_V3:SAMTEC_TSW-105-08-G-T-RA, symbol 5x15Conn:TSW-105-08-G-T-RA
- added J11, J13, J4: Conn_01x04, Connector_Molex:Molex_PicoBlade_53048-0410_1x04_P1.25mm_Horizontal, symbol Connector_Generic:Conn_01x04
- added J12, J8: Conn_01x02, Connector_PinHeader_2.54mm:PinHeader_1x02_P2.54mm_Vertical, symbol Connector_Generic:Conn_01x02
- added J14: Conn_02x04_Odd_Even, Connector_PinHeader_2.54mm:PinHeader_2x04_P2.54mm_Vertical_SMD, symbol Connector_Generic:Conn_02x04_Odd_Even
- added J15: Conn_01x02, Connector_PinHeader_2.54mm:PinHeader_1x02_P2.54mm_Vertical_SMD_Pin1Left, symbol Connector_Generic:Conn_01x02
- added J16, J2, J7: Conn_01x02, Connector_Molex:Molex_Mega-Fit_76825-0002_2x01_P5.70mm_Horizontal, symbol Connector_Generic:Conn_01x02
- added J19: Conn_02x02_Odd_Even, Connector_PinHeader_2.54mm:PinHeader_2x02_P2.54mm_Vertical, symbol Connector_Generic:Conn_02x02_Odd_Even
- added J3: Conn_01x02, Connector_Molex:Molex_Micro-Fit_3.0_43045-0200_2x01_P3.00mm_Horizontal, symbol Connector_Generic:Conn_01x02
- added R1: 3000, Resistor_SMD:R_0805_2012Metric_Pad1.20x1.40mm_HandSolder, symbol Device:R
- added R2: 750, Resistor_SMD:R_0805_2012Metric_Pad1.20x1.40mm_HandSolder, symbol Device:R
- added R3: 150, Resistor_SMD:R_0805_2012Metric_Pad1.20x1.40mm_HandSolder, symbol Device:R
- added R4: 976, Resistor_SMD:R_0805_2012Metric_Pad1.20x1.40mm_HandSolder, symbol Device:R
- added U2: LED8102SXTTR, ManipulatorER_V3:LED8102SXTTR, symbol LED_IC:LED8102SXTTR
- C1: value C -> 0.1u; footprint Ceramic:C1206C104J4RAC7800 -> ManipulatorER_V3:C1206C104J4RAC7800
- C3: footprint Ele Caps:UCM1H220MCL1GS -> ManipulatorER_V3:UCM1H220MCL1GS
- J1: footprint Connector_Dsub:DSUB-15_Female_Horizontal_P2.77x2.84mm_EdgePinOffset4.94mm_Housed_MountingHolesOffset7.48mm -> Connector_Dsub:DSUB-15_Female_Horizontal_P2.77x2.84mm_EdgePinOffset7.70mm_Housed_MountingHolesOffset9.12mm
- J6: footprint Connector_Molex:Molex_Micro-Fit_3.0_43045-0400_2x02_P3.00mm_Horizontal -> Connector_Molex:Molex_PicoBlade_53048-0410_1x04_P1.25mm_Horizontal
- P1: footprint Socket_Arduino_Mega:Socket_Strip_Arduino_2x18 -> ManipulatorER_V3:Socket_Strip_Arduino_2x18
- P2, P3, P4, P6, P7: footprint Socket_Arduino_Mega:Socket_Strip_Arduino_1x08 -> ManipulatorER_V3:Socket_Strip_Arduino_1x08
- P5: footprint Socket_Arduino_Mega:Socket_Strip_Arduino_1x10 -> ManipulatorER_V3:Socket_Strip_Arduino_1x10
- U1: footprint TS Regulators:TSR 1-2433 -> ManipulatorER_V3:TSR 1-2433
- renumbered J1001 to J17
Connections:
- net Vin is gone; now on net +5V: P2.8 (Pin_8)
- net +5V: now also D1.2 (A), D2.2 (A), D3.2 (A), D4.2 (A), J11.4 (Pin_4), J13.4 (Pin_4), J14.2 (Pin_2), J14.4 (Pin_4), J14.6 (Pin_6), J14.8 (Pin_8), J19.3 (Pin_3), J3.2 (Pin_2), J4.4 (Pin_4), R3.2, U2.16 (VDD)
- net 0(Rx0): now also J15.2 (Pin_2), U2.4 (SW3)
- net 1(Tx0): now also J15.1 (Pin_1), U2.13 (SW4)
- net 10(**): now also J10.02
- net 12V: now also C3.1, U1.1 (Vin), C4.2, J2.2 (Pin_2), J7.2 (Pin_2), R2.2
- net 16(Tx2): now also J4.2 (Pin_2)
- net 17(Rx2): now also J4.3 (Pin_3)
- net 20(SDA): now also J6.3 (Pin_3)
- net 21(SCL): now also J6.4 (Pin_4)
- net 23: now also J10.13
- net 25: now also J10.10
- net 27: now also J10.14; no longer J6.3 (Pin_3)
- net 29: now also J10.11; no longer J6.4 (Pin_4)
- net 31: now also J10.15
- net 32: now also J10.12
- net 37: now also J9.14
- net 39: now also J9.11
- net 3V3: now also P2.4 (Pin_4)
- net 40: now also J9.13
- net 40V: now also J12.2 (Pin_2), J8.2 (Pin_2), R1.2; no longer C3.1, U1.1 (Vin)
- net 41: now also J9.10
- net 42: now also J9.15
- net 43: now also J9.12
- net 44: now also J9.01
- net 45: now also J9.02
- net 46: now also J10.01
- net 47: now also U2.3 (SW2)
- net 49: now also U2.2 (SW1)
- net 50(MISO): now also J11.2 (Pin_2)
- net 51(MOSI): now also J11.3 (Pin_3)
- net 52(SCK): now also J13.2 (Pin_2)
- net 53(SS): now also J13.3 (Pin_3)
- net 7(**): now also J9.03
- net 9(**): now also J10.03
- net A10: now also J1.12 (P12)
- net A11: now also J1.4; no longer J1.11 (P111)
- net A12: now also J1.11 (P111); no longer J1.4
- net A13: no longer J1.12 (P12)
- net A14: no longer J1.5
- net A15: no longer J1.13 (P13)
- net A5: now also J1.13 (P13)
- net A9: now also J1.5
- net GND: now also C4.1, D5.1 (K), D6.1 (K), D7.1 (K), J10.07, J10.08, J10.09, J11.1 (Pin_1), J12.1 (Pin_1), J13.1 (Pin_1), J16.1 (Pin_1), J2.1 (Pin_1), J3.1 (Pin_1), J4.1 (Pin_1), J7.1 (Pin_1), J8.1 (Pin_1), J9.07, J9.08, J9.09, R4.2, U2.1 (GND), U2.14 (*OE), U2.EPAD (GND)
- net SCL renamed 1
- net SDA renamed 2
- new net: D7.2 (A), R3.1
- new net: D6.2 (A), R2.1
- new net: D5.2 (A), R1.1
- new net: D1.1 (K), U2.5 (OUT0)
- new net: D2.1 (K), U2.7 (OUT2)
- new net: D4.1 (K), U2.11 (OUT6)
- new net: J14.5 (Pin_5), U2.10 (OUT5)
- new net: J14.7 (Pin_7), U2.12 (OUT7)
- new net: R4.1, U2.15 (R-EXT)
- new net: J14.1 (Pin_1), U2.6 (OUT1)
- new net: J14.3 (Pin_3), U2.8 (OUT3)
- new net: D3.1 (K), U2.9 (OUT4)
- new net +7V: J16.2 (Pin_2), J19.1 (Pin_1)
- new net Vmisc: J10.04, J10.05, J10.06, J19.2 (Pin_2), J19.4 (Pin_4), J9.04, J9.05, J9.06
- no-connect marks 4 -> 3
Other:
- moved on the sheet: C1, J5
