File: Payload_PCB_v3.1.kicad_sch (KiCad schematic)
At the start: 194 parts, among them J1 Power Input, J10 DB9 - Analog Inputs, J11 DB25 - IO and Payload Select, J12 DB37 Connector, J13 USB2CAN, J14 CAN1, J15 CAN2, J16 Terminator, J17 Terminator, J18 USB_B_Micro, J2 Power Output, J3 40V jumper, J4 Vmisc Select, J5 Conn_01x04, J6 Conn_01x04, J7 Conn_01x04, J8 Conn_01x04, J9 Extra IO, Q1 SUD50P10-43L-GE3, Q2 SUD50P10-43L-GE3, Q3 SUD50P10-43L-GE3, Q4 DMG2305UX, U1 ROB-14450, U10 PCA9555PWR, U11 VCB4812SBO-100WR3-N, U12 TSR 2-2450, U13 MCP3428, U14 Pico, U15 74HCT244, U16 PCA9685PW, U17 LED8102SXTTR, U18 74HCT244, U19 ISO1050DUB, U2 ROB-14450, U20 RT9080-33GJ5, U21 B0505S, U22 MCP2562, U23 MCP2515, U3 DRV8874, U4 DRV8874, U5 DRV8874, U6 DRV8874, U7 PCA9555PWR, U8 PCA9555PWR, U9 TSR 2-2433, Y1 8 MHz

Commit message: initial cleanup of repo
Parts:
- C1: value 0.1 uF -> 0.1 uF
Other:
- note added: "5V is jumpered to Vsel on the PCB in Science"
- note added: "CHANGE FROM +3V3 to +5 RELABEL PINS BASED OFF EVERYTHING ELSE"
- note added: "KEEP JUST IN CASE"
- note added: "MAKE THE U2D2 PLUG IN VIA BARREL CONNECTOR ADD BREAKOUTS FOR I2C CONNECTIONS IN CASE WE WANT OTHER THINGS OR SENSORS"
- note added: "POTS ARE MOISTURE AND TEMPERATURE. ONE IS UNUSED/LOOPED BACK TO ANOTHER PIN. THE BIG CONNECTOR CONNECTS TO 2 RELAYS"
- note added: "SCIENCE: 3V3 is jumpered from pin 2 to pin 8 Pin 3 to temp sensor with power +3V3 Pin 7 to moisture with +3V3"
- note added: "SCIENCE: P_S1 is floating taped. GP21 to closer relay = 12V ? GP22 to further relay = 12V ?"
- note added: "SCIENCE: servo 1-4 are used on science Pin 7 = scoop 1 Pin 26 = scoop 2 Pin 8 and 27 = connector"
- note added: "THIS HAS 2 PER POWER/GROUND AND 4 SERVO CONNECTIONS."
- note added: "THIS IS RARELY POPULATED, AND WHEN IT IS, THE USB PORT ISN'T, MEANING THAT IT DOESN'T CONNECT TO ANYTHING REMOVE IF UNUSED BY MANIPULATION"
- note added: "TODO"
- note added: "WHY DO WE TAKE IN 40V, WHY NOT JUST USE THE 12V WE ARE GIVEN TO POWER EVERYTHING AND GET RID OF U11 COMPLETELY"
