File: leds.kicad_sch (KiCad schematic)
At the start: 28 parts, among them Q5 Q_NMOS, Q6 Q_NMOS, Q7 Q_NMOS, Q8 Q_NMOS

Commit message: more cleanup and added notes for review
Other:
- moved on the sheet: D4, D5, D6, D7, D8, R15, R16, R17, R18, R19, R20, R21

Commit message: pcb review session notes
Other:
- moved on the sheet: D10, D11, D12, D9
Changed lines of the file:
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@@
 	(wire
 		(pts
-			(xy 215.9 102.87) (xy 208.28 102.87)
+			(xy 212.09 102.87) (xy 208.28 102.87)
 		)
 		(stroke
@@
 	(wire
 		(pts
-			(xy 223.52 102.87) (xy 227.33 102.87)
+			(xy 219.71 102.87) (xy 227.33 102.87)
 		)
 		(stroke
@@
 	(wire
 		(pts
-			(xy 223.52 86.36) (xy 227.33 86.36)
+			(xy 219.71 86.36) (xy 227.33 86.36)
 		)
 		(stroke
@@
 	(wire
 		(pts
-			(xy 223.52 119.38) (xy 227.33 119.38)
+			(xy 219.71 119.38) (xy 227.33 119.38)
 		)
 		(stroke
@@
 	(wire
 		(pts
-			(xy 215.9 86.36) (xy 208.28 86.36)
+			(xy 212.09 86.36) (xy 208.28 86.36)
 		)
 		(stroke
@@
 	(wire
 		(pts
-			(xy 215.9 69.85) (xy 208.28 69.85)
+			(xy 212.09 69.85) (xy 208.28 69.85)
 		)
 		(stroke
@@
 	(wire
 		(pts
-			(xy 227.33 69.85) (xy 223.52 69.85)
+			(xy 227.33 69.85) (xy 219.71 69.85)
 		)
 		(stroke
@@
 	(wire
 		(pts
-			(xy 215.9 119.38) (xy 208.28 119.38)
+			(xy 212.09 119.38) (xy 208.28 119.38)
 		)
 		(stroke
@@
 	(symbol
 		(lib_id "Device:LED")
-		(at 219.71 69.85 180)
+		(at 215.9 69.85 180)
 		(unit 1)
 		(exclude_from_sim no)
@@
 		(dnp no)
 		(property "Reference" "D9"
-			(at 217.424 65.786 0)
+			(at 213.614 65.786 0)
 			(effects
 				(font
@@
 		)
 		(property "Value" "LED1"
-			(at 222.758 65.786 0)
+			(at 218.948 65.786 0)
 			(effects
 				(font
@@
 		)
 		(property "Footprint" "LED_SMD:LED_0805_2012Metric_Pad1.15x1.40mm_HandSolder"
-			(at 219.71 69.85 0)
+			(at 215.9 69.85 0)
 			(effects
 				(font
@@
 		)
 		(property "Datasheet" "~"
-			(at 219.71 69.85 0)
+			(at 215.9 69.85 0)
 			(effects
 				(font
@@
 		)
 		(property "Description" ""
-			(at 219.71 69.85 0)
+			(at 215.9 69.85 0)
 			(effects
 				(font
@@
 		)
 		(property "Manufacturer" ""
-			(at 219.71 69.85 0)
+			(at 215.9 69.85 0)
 			(effects
 				(font
@@
 		)
 		(property "Manufacturer Part Number" ""
-			(at 219.71 69.85 0)
+			(at 215.9 69.85 0)
 			(effects
 				(font
@@
 		)
 		(property "Vendor" ""
-			(at 219.71 69.85 0)
+			(at 215.9 69.85 0)
 			(effects
 				(font
@@
 		)
 		(property "Vendor Part Number" ""
-			(at 219.71 69.85 0)
+			(at 215.9 69.85 0)
 			(effects
 				(font
@@
 		)
 		(property "Comments" ""
-			(at 219.71 69.85 0)
+			(at 215.9 69.85 0)
 			(effects
 				(font
@@
 		)
 		(property "Notes" ""
-			(at 219.71 69.85 0)
+			(at 215.9 69.85 0)
 			(effects
 				(font
@@
 	(symbol
 		(lib_id "Device:LED")
-		(at 219.71 102.87 180)
+		(at 215.9 102.87 180)
 		(unit 1)
 		(exclude_from_sim no)
@@
 		(dnp no)
 		(property "Reference" "D12"
-			(at 217.424 98.806 0)
+			(at 213.614 98.806 0)
 			(effects
 				(font
@@
 		)
 		(property "Value" "LED3"
-			(at 222.758 98.806 0)
+			(at 218.948 98.806 0)
 			(effects
 				(font
@@
 		)
 		(property "Footprint" "LED_SMD:LED_0805_2012Metric_Pad1.15x1.40mm_HandSolder"
-			(at 219.71 102.87 0)
+			(at 215.9 102.87 0)
 			(effects
 				(font
@@
 		)
 		(property "Datasheet" "~"
-			(at 219.71 102.87 0)
+			(at 215.9 102.87 0)
 			(effects
 				(font
@@
 		)
 		(property "Description" ""
-			(at 219.71 102.87 0)
+			(at 215.9 102.87 0)
 			(effects
 				(font
@@
 		)
 		(property "Manufacturer" ""
-			(at 219.71 102.87 0)
+			(at 215.9 102.87 0)
 			(effects
 				(font
@@
 		)
 		(property "Manufacturer Part Number" ""
-			(at 219.71 102.87 0)
+			(at 215.9 102.87 0)
 			(effects
 				(font
@@
 		)
 		(property "Vendor" ""
-			(at 219.71 102.87 0)
+			(at 215.9 102.87 0)
 			(effects
 				(font
@@
 		)
 		(property "Vendor Part Number" ""
-			(at 219.71 102.87 0)
+			(at 215.9 102.87 0)
 			(effects
 				(font
@@
 		)
 		(property "Comments" ""
-			(at 219.71 102.87 0)
+			(at 215.9 102.87 0)
 			(effects
 				(font
@@
 		)
 		(property "Notes" ""
-			(at 219.71 102.87 0)
+			(at 215.9 102.87 0)
 			(effects
 				(font
@@
 	(symbol
 		(lib_id "Device:LED")
-		(at 219.71 119.38 180)
+		(at 215.9 119.38 180)
 		(unit 1)
 		(exclude_from_sim no)
@@
 		(dnp no)
 		(property "Reference" "D11"
-			(at 217.424 115.316 0)
+			(at 213.614 115.316 0)
 			(effects
 				(font
@@
 		)
 		(property "Value" "LED4"
-			(at 222.758 115.316 0)
+			(at 218.948 115.316 0)
 			(effects
 				(font
@@
 		)
 		(property "Footprint" "LED_SMD:LED_0805_2012Metric_Pad1.15x1.40mm_HandSolder"
-			(at 219.71 119.38 0)
+			(at 215.9 119.38 0)
 			(effects
 				(font
@@
 		)
 		(property "Datasheet" "~"
-			(at 219.71 119.38 0)
+			(at 215.9 119.38 0)
 			(effects
 				(font
@@
 		)
 		(property "Description" ""
-			(at 219.71 119.38 0)
+			(at 215.9 119.38 0)
 			(effects
 				(font
@@
 		)
 		(property "Manufacturer" ""
-			(at 219.71 119.38 0)
+			(at 215.9 119.38 0)
 			(effects
 				(font
@@
 		)
 		(property "Manufacturer Part Number" ""
-			(at 219.71 119.38 0)
+			(at 215.9 119.38 0)
 			(effects
 				(font
@@
 		)
 		(property "Vendor" ""
-			(at 219.71 119.38 0)
+			(at 215.9 119.38 0)
 			(effects
 				(font
@@
 		)
 		(property "Vendor Part Number" ""
-			(at 219.71 119.38 0)
+			(at 215.9 119.38 0)
 			(effects
 				(font
@@
 		)
 		(property "Comments" ""
-			(at 219.71 119.38 0)
+			(at 215.9 119.38 0)
 			(effects
 				(font
@@
 		)
 		(property "Notes" ""
-			(at 219.71 119.38 0)
+			(at 215.9 119.38 0)
 			(effects
 				(font
@@
 	(symbol
 		(lib_id "Device:LED")
-		(at 219.71 86.36 180)
+		(at 215.9 86.36 180)
 		(unit 1)
 		(exclude_from_sim no)
@@
 		(dnp no)
 		(property "Reference" "D10"
-			(at 217.424 82.296 0)
+			(at 213.614 82.296 0)
 			(effects
 				(font
@@
 		)
 		(property "Value" "LED2"
-			(at 222.758 82.296 0)
+			(at 218.948 82.296 0)
 			(effects
 				(font
@@
 		)
 		(property "Footprint" "LED_SMD:LED_0805_2012Metric_Pad1.15x1.40mm_HandSolder"
-			(at 219.71 86.36 0)
+			(at 215.9 86.36 0)
 			(effects
 				(font
@@
 		)
 		(property "Datasheet" "~"
-			(at 219.71 86.36 0)
+			(at 215.9 86.36 0)
 			(effects
 				(font
@@
 		)
 		(property "Description" ""
-			(at 219.71 86.36 0)
+			(at 215.9 86.36 0)
 			(effects
 				(font
@@
 		)
 		(property "Manufacturer" ""
-			(at 219.71 86.36 0)
+			(at 215.9 86.36 0)
 			(effects
 				(font
@@
 		)
 		(property "Manufacturer Part Number" ""
-			(at 219.71 86.36 0)
+			(at 215.9 86.36 0)
 			(effects
 				(font
@@
 		)
 		(property "Vendor" ""
-			(at 219.71 86.36 0)
+			(at 215.9 86.36 0)
 			(effects
 				(font
@@
 		)
 		(property "Vendor Part Number" ""
-			(at 219.71 86.36 0)
+			(at 215.9 86.36 0)
 			(effects
 				(font
@@
 		)
 		(property "Comments" ""
-			(at 219.71 86.36 0)
+			(at 215.9 86.36 0)
 			(effects
 				(font
@@
 		)
 		(property "Notes" ""
-			(at 219.71 86.36 0)
+			(at 215.9 86.36 0)
 			(effects
 				(font

Commit message: major rework again after the meeting
Parts:
- removed D10: LED2, LED_SMD:LED_0805_2012Metric_Pad1.15x1.40mm_HandSolder, symbol Device:LED
- removed D11: LED4, LED_SMD:LED_0805_2012Metric_Pad1.15x1.40mm_HandSolder, symbol Device:LED
- removed D12: LED3, LED_SMD:LED_0805_2012Metric_Pad1.15x1.40mm_HandSolder, symbol Device:LED
- removed D4: +40V, LED_SMD:LED_0805_2012Metric_Pad1.15x1.40mm_HandSolder, symbol Device:LED
- removed D5: +12V, LED_SMD:LED_0805_2012Metric_Pad1.15x1.40mm_HandSolder, symbol Device:LED
- removed D6: VDC, LED_SMD:LED_0805_2012Metric_Pad1.15x1.40mm_HandSolder, symbol Device:LED
- removed D7: +5V, LED_SMD:LED_0805_2012Metric_Pad1.15x1.40mm_HandSolder, symbol Device:LED
- removed D8: +3V3, LED_SMD:LED_0805_2012Metric_Pad1.15x1.40mm_HandSolder, symbol Device:LED
- removed D9: LED1, LED_SMD:LED_0805_2012Metric_Pad1.15x1.40mm_HandSolder, symbol Device:LED
- removed Q5, Q6, Q7, Q8: Q_NMOS, Package_TO_SOT_SMD:TSOT-23, symbol Transistor_FET:Q_NMOS_DGS
- removed R1, R17, R5, R6, R8: 511, Resistor_SMD:R_0805_2012Metric_Pad1.20x1.40mm_HandSolder, symbol Device:R_US
- removed R15, R20: 1k, Resistor_SMD:R_0805_2012Metric_Pad1.20x1.40mm_HandSolder, symbol Device:R_US
- removed R16, R18, R21: 150, Resistor_SMD:R_0805_2012Metric_Pad1.20x1.40mm_HandSolder, symbol Device:R_US
- removed R19: 62, Resistor_SMD:R_0805_2012Metric_Pad1.20x1.40mm_HandSolder, symbol Device:R_US
- removed TP12: LED1, TestPoint:TestPoint_Pad_D1.0mm, symbol Connector:TestPoint
- removed TP13: LED2, TestPoint:TestPoint_Pad_D1.0mm, symbol Connector:TestPoint
- removed TP14: LED4, TestPoint:TestPoint_Pad_D1.0mm, symbol Connector:TestPoint
- removed TP16: LED3, TestPoint:TestPoint_Pad_D1.0mm, symbol Connector:TestPoint
Other:
- note removed: "DEVELOPMENT LEDs"
- note removed: "POWER LEDs"
