File: payload-pcb.kicad_pcb (KiCad board)
At the start: 4 copper layers, 127 x 76.2 mm, 100 parts, among them J1 POWER_IN, J10 QWIIC3, J11 QWIIC2, J12 I2C, J13 QWIIC1, J14 CAN, J15 CAN, J16 SERVO4, J17 SERVO3, J18 MANIPULATOR, J19 SCOOP, J2 POWER_OUT, J20 EXP1, J21 EXP2, J22 EXP3, J23 EXP4, J3 UART, J4 USB, J5 MST, J6 TMP, J7 MPR, J8 QWIIC4, J9 DIGITAL, Q1 SUD50P10-43L-GE3, Q2 MMBT3904, Q4 DMG2305UX, Q5 2N7002, Q6 2N7002, SW1 QUIIC, SW2 EXP, U1 SN74AHCT126DR, U12 +3V3@2A, U14 PI_PICO, U2 FT230XS, U22 MCP2562, U23 MCP2515, U3 LTC2990, U9 +5V@2A, Y1 8MHz

Commit message: swapped UART to USB from FTDI (out of stock) to MCP2200
Parts:
- removed C30, C31: 22pF, Capacitor_SMD:C_0603_1608Metric_Pad1.08x0.95mm_HandSolder
- removed U2: FT230XS, Package_SO:SSOP-16_3.9x4.9mm_P0.635mm
- added C11: 12pF, Capacitor_SMD:C_0603_1608Metric_Pad1.08x0.95mm_HandSolder, F.Cu at (172.8, 80.0)
- added C12: 12pF, Capacitor_SMD:C_0603_1608Metric_Pad1.08x0.95mm_HandSolder, F.Cu at (170.4, 77.3)
- added C13: 0.1uF, Capacitor_SMD:C_1206_3216Metric_Pad1.33x1.80mm_HandSolder, F.Cu at (165.0, 72.2)
- added C14: 12pF, Capacitor_SMD:C_0603_1608Metric_Pad1.08x0.95mm_HandSolder, F.Cu at (157.6, 133.1)
- added C15: 12pF, Capacitor_SMD:C_0603_1608Metric_Pad1.08x0.95mm_HandSolder, F.Cu at (154.6, 135.7)
- added D4: TX, LED_SMD:LED_0805_2012Metric_Pad1.15x1.40mm_HandSolder, F.Cu at (149.6, 77.8)
- added D6: RX, LED_SMD:LED_0805_2012Metric_Pad1.15x1.40mm_HandSolder, F.Cu at (149.6, 79.9)
- added R18: 10k, Resistor_SMD:R_0603_1608Metric_Pad0.98x0.95mm_HandSolder, F.Cu at (162.6, 76.6)
- added R19: 330, Resistor_SMD:R_0603_1608Metric_Pad0.98x0.95mm_HandSolder, F.Cu at (146.1, 77.8)
- added R20: 22, Resistor_SMD:R_0603_1608Metric_Pad0.98x0.95mm_HandSolder, F.Cu at (146.1, 79.9)
- added TP4: +5V, TestPoint:TestPoint_Pad_D2.0mm, F.Cu at (113.6, 71.5)
- added TP6: +3V3, TestPoint:TestPoint_Pad_D2.0mm, F.Cu at (167.6, 90.3)
- added U4: MCP2200, Package_SO:SSOP-20_5.3x7.2mm_P0.65mm, F.Cu at (162.6, 81.3)
- added Y3: 12MHz, Crystal:Crystal_SMD_2520-4Pin_2.5x2.0mm, F.Cu at (170.4, 80.0)
- C2, C3, C8: footprint Capacitor_SMD:C_1206_3216Metric_Pad1.33x1.80mm_HandSolder -> Capacitor_SMD:C_0805_2012Metric_Pad1.18x1.45mm_HandSolder
- C9: value 470p -> 470pF
- R1, R3: value 511 -> 22
- R17: value 511 -> 1k78
- R22, R23: value 3.3k -> 3k3
- R4, R5: value 511 -> 330
- Y1: footprint Crystal:Crystal_SMD_HC49-SD -> Crystal:Crystal_SMD_3225-4Pin_3.2x2.5mm
- moved C3 10.3 mm to (162.6, 86.3)
- moved C8 6.21 mm to (156.8, 80.6), turned to 90 degrees
- moved Y1 1.94 mm to (157.6, 135.7), turned to 180 degrees
- moved R3 1.65 mm to (98.4, 106.8)
- moved R4 1.65 mm to (98.4, 105.2)
- turned R5 to -90 degrees
Connections:
- net /Pi Pico/LED_BAD renamed /Pi Pico/LED_ERROR
- net /Pi Pico/LED_GOOD renamed /Pi Pico/LED_STATUS
- C8 pad 1: GND -> /USB/+V_USB
- C8 pad 2: Net-(U2-3V3OUT) -> GND
- R3 pad 1: Net-(D2-A) -> Net-(D3-A)
- R3 pad 2: +5V -> +3V3
- R4 pad 1: Net-(D3-A) -> Net-(D2-A)
- R4 pad 2: +3V3 -> +5V
- R5 pad 1: Net-(D10-A) -> +3V3
- R5 pad 2: +3V3 -> Net-(D10-A)
- R6 pad 2: /USB/USB_OUT- -> /USB/USB_OUT+
- R7 pad 2: /USB/USB_OUT+ -> /USB/USB_OUT-
- Y1 pad 1: Net-(U23-OSC1) -> Net-(U23-OSC2)
- Y1 pad 2: Net-(U23-OSC2) -> GND
Routing:
- net +3V3: track 211.3 -> 228.7 mm, vias 27 -> 29
- net Net-(D4-K): track 0.00 -> 16.8 mm, vias 0 -> 2
- net Net-(D6-K): track 0.00 -> 16.2 mm, vias 0 -> 2
- net Net-(U2-3V3OUT): track 14.9 -> 0.00 mm, vias 2 -> 0
- net +5V: track 46.2 -> 56.9 mm
- net Net-(U4-OSC2): track 0.00 -> 8.39 mm
- net /GPIO/+QUIIC: track 114.7 -> 123.0 mm, vias 4 -> 7
- net Net-(U4-OSC1): track 0.00 -> 8.27 mm
- net Net-(U4-RST): track 0.00 -> 7.97 mm
- net GND: track 46.1 -> 51.9 mm, vias 190 -> 218
- net Net-(U23-OSC2): track 13.4 -> 8.35 mm
- net /USB/USB_OUT+: track 13.1 -> 9.06 mm
- net /USB/USB_OUT-: track 13.1 -> 9.09 mm
- net UART0_RX: track 36.1 -> 32.1 mm
- net /USB/+V_USB: track 0.00 -> 2.49 mm
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Other:
- board text added: "TX RX"

Commit message: added release documents for v5.1 (pending approval)
Parts:
- renumbered Y3 to Y2
Changed lines of the file:
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@@
 	(paper "A4")
 	(title_block
-		(date "mar. 31 mars 2015")
+		(title "Payload PCB")
+		(date "2026-01-03")
+		(rev "v5.1")
+		(company "WVU Unviersity Rover Challenge (URC)")
 	)
 	(layers
@@
 		(at 170.3832 79.9592 90)
 		(descr "SMD2520/4, Crystal, 2.5x2.0mm package, SMD, generated with kicad-footprint-generator make_crystal.py, http://www.newxtal.com/UploadFiles/Images/2012-11-12-09-29-09-776.pdf")
-		(property "Reference" "Y3"
+		(property "Reference" "Y2"
 			(at -2.3622 0.8382 180)
 			(layer "F.SilkS")

Commit message: touch ups from peer reviews
Parts:
- added C16: 0.1uF, Capacitor_SMD:C_0805_2012Metric_Pad1.18x1.45mm_HandSolder, F.Cu at (146.9, 69.6)
- added U2: MIC94093YC6, Package_TO_SOT_SMD:SOT-363_SC-70-6, F.Cu at (146.9, 73.0)
- moved C2 1.00 mm to (160.7, 72.1), turned to 90 degrees
Connections:
- C2 pad 2: +5V -> +VBUS
- J4 pad 1: +5V -> +VBUS
- R6 pad 2: /USB/USB_OUT+ -> /USB/USB_OUT-
- R7 pad 2: /USB/USB_OUT- -> /USB/USB_OUT+
- U4 pad 18: /USB/USB_OUT+ -> /USB/USB_OUT-
- U4 pad 19: /USB/USB_OUT- -> /USB/USB_OUT+
Routing:
- net +VBUS: track 0.00 -> 27.7 mm, vias 0 -> 9
- net +5V: track 56.9 -> 59.4 mm
- net GND: track 51.9 -> 53.5 mm, vias 218 -> 221
- added copper zone on B.Cu, net +VBUS
- added copper zone on F.Cu, net +VBUS
