File: payload-pcb.kicad_pcb (KiCad board)
At the start: 4 copper layers, 127 x 76.2 mm, 113 parts, among them J1 POWER_IN, J10 QWIIC3, J11 QWIIC2, J12 I2C, J13 QWIIC1, J14 CAN, J15 CAN, J16 SERVO4, J17 SERVO3, J18 MANIPULATOR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

Commit message: schematic cleanup
Parts:
- added REF**: OSHW-Logo_7.5x8mm_SilkScreen, Symbol:OSHW-Logo_7.5x8mm_SilkScreen, F.Cu at (182.1, 137.0)
