File: gpio.kicad_sch (KiCad schematic)
At the start: 29 parts, among them J10 QWIIC3, J11 QWIIC2, J13 QWIIC1, J16 SERVO4, J17 SERVO3, J18 MANIPULATOR, J19 SCOOP, J20 EXP1, J21 EXP2, J22 EXP3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

Commit message: Added housing/cable/header info to each connector's symbol properties.
Parts:
- J16, J17, J18, J19, J5, J6, J7: Cable (none) -> 0500798000-06-B6; Housing (none) -> 0510210300
- J9: Cable (none) -> 0500798000-06-B6; Housing (none) -> 0510210800
