File: power.kicad_sch (KiCad schematic)
At the start: 31 parts, among them J1 POWER_IN, J2 POWER_OUT, Q1 SUD50P10-43L-GE3, Q2 MMBT3904, U12 +3V3@2A, U3 LTC2990, U9 +5V@2A

Commit message: Added housing/cable/header info to each connector's symbol properties.
Parts:
- J1: Assembly (none) -> 2147561021
- J2: Assembly (none) -> 2147561061
