File: power.kicad_sch (KiCad schematic)
At the start: 31 parts, among them J1 POWER_IN, J2 POWER_OUT, Q1 SUD50P10-43L-GE3, Q2 MMBT3904, U12 +3V3@2A, U3 LTC2990, U9 +5V@2A

Commit message: schematic cleanup
Changed lines of the file:
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@@
 	(text "7-bit = 0x4C\nRead = 0x99\nWrite = 0x98"
 		(exclude_from_sim no)
-		(at 135.89 95.25 0)
+		(at 131.572 93.472 0)
 		(effects
 			(font
