File: payload-pcb.kicad_sch (KiCad schematic)
At the start: 4 parts

Commit message: schematic cleanup
Other:
- note added: "URC Payload PCB"
- note removed: "Payload PCB"
- title: Payload PCB -> URC Payload PCB
Changed lines of the file:
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@@
 	(paper "A4")
 	(title_block
-		(title "Payload PCB")
+		(title "URC Payload PCB")
 		(date "2026-01-16")
 		(rev "v5.1")
 		(company "WVU Unviersity Rover Challenge (URC)")
 	)
-	(text "Payload PCB"
-		(exclude_from_sim no)
-		(at 148.59 34.29 0)
+	(text "URC Payload PCB"
+		(exclude_from_sim no)
+		(at 149.86 33.02 0)
 		(effects
 			(font
@@
 	(text "by Austin Driggs\n2025-2026"
 		(exclude_from_sim no)
-		(at 148.59 43.434 0)
+		(at 149.86 43.18 0)
 		(effects
 			(font
@@
 		)
 	)
+	(polyline
+		(pts
+			(xy 118.364 37.846) (xy 181.864 37.846)
+		)
+		(stroke
+			(width 0)
+			(type default)
+		)
+	)
 	(symbol
 		(lib_name "MountingHole_Pad_2")
@@
 				)
 				(justify left)
+				(hide yes)
 			)
 		)
@@
 				)
 				(justify left)
+				(hide yes)
 			)
 		)
@@
 				)
 				(justify left)
+				(hide yes)
 			)
 		)
@@
 				)
 				(justify left)
+				(hide yes)
 			)
 		)
@@
 					(unit 1)
 				)
+			)
+		)
+	)
+	(symbol
+		(lib_id "Graphic:Logo_Open_Hardware_Large")
+		(at 160.02 182.88 0)
+		(unit 1)
+		(exclude_from_sim no)
+		(in_bom no)
+		(on_board no)
+		(dnp no)
+		(fields_autoplaced yes)
+		(property "Reference" "#SYM1"
+			(at 160.02 170.18 0)
+			(effects
+				(font
+					(size 1.27 1.27)
+				)
+				(hide yes)
+			)
+		)
+		(property "Value" "Logo_Open_Hardware_Large"
+			(at 160.02 193.04 0)
+			(effects
+				(font
+					(size 1.27 1.27)
+				)
+				(hide yes)
+			)
+		)
+		(property "Footprint" ""
+			(at 160.02 182.88 0)
+			(effects
+				(font
+					(size 1.27 1.27)
+				)
+				(hide yes)
+			)
+		)
+		(property "Datasheet" "~"
+			(at 160.02 182.88 0)
+			(effects
+				(font
+					(size 1.27 1.27)
+				)
+				(hide yes)
+			)
+		)
+		(property "Description" "Open Hardware logo, large"
+			(at 160.02 182.88 0)
+			(effects
+				(font
+					(size 1.27 1.27)
+				)
+				(hide yes)
+			)
+		)
+		(instances
+			(project ""
+				(path "/29e78086-2175-405e-9ba3-c48766d2f50c"
+					(reference "#SYM1")
+					(unit 1)
+				)
